Commit message: add robot description

File: src/rail_robot/urdf/battery.urdf.xacro (robot description, xacro)
@@ -5,9 +5,9 @@
       <xacro:insert_block name="origin"/>
       <parent
-        link="plate_link"/>
+        link="${robot_name}/plate_link"/>
       <child
-        link="battery_link"/>
+        link="${robot_name}/battery_link"/>
     </joint>
-    <link name="battery_link">
+    <link name="${robot_name}/battery_link">
       <visual>
         <origin
@@ -48,5 +48,5 @@
       </inertial>
     </link>
-    <gazebo reference="battery_link">
+    <gazebo reference="${robot_name}/battery_link">
       <material>Gazebo/Grey</material>
     </gazebo>

File: src/rail_robot/urdf/camera_tower.urdf.xacro (robot description, xacro)
@@ -5,9 +5,9 @@
       <xacro:insert_block name="origin"/>
       <parent
-        link="base_link"/>
+        link="${robot_name}/base_link"/>
       <child
-        link="camera_tower_link"/>
+        link="${robot_name}/camera_tower_link"/>
     </joint>
-    <link name="camera_tower_link">
+    <link name="${robot_name}/camera_tower_link">
       <visual>
         <origin
@@ -33,5 +33,5 @@
       <xacro:insert_block name="inertial"/>
     </link>
-    <gazebo reference="camera_tower_link">
+    <gazebo reference="${robot_name}/camera_tower_link">
       <material>Gazebo/DarkGrey</material>
     </gazebo>

File: src/rail_robot/urdf/lidar.urdf.xacro (robot description, xacro)
@@ -5,9 +5,9 @@
       <xacro:insert_block name="origin"/>
       <parent
-        link="camera_tower_link"/>
+        link="${robot_name}/camera_tower_link"/>
       <child
-        link="lidar_tower_link"/>
+        link="${robot_name}/lidar_tower_link"/>
     </joint>
-    <link name="lidar_tower_link">
+    <link name="${robot_name}/lidar_tower_link">
       <visual>
         <origin
@@ -50,9 +50,9 @@
         xyz="0 0 0.09425"/>
       <parent
-        link="lidar_tower_link"/>
+        link="${robot_name}/lidar_tower_link"/>
       <child
-        link="laser_frame_link"/>
+        link="${robot_name}/laser_frame_link"/>
     </joint>
-    <link name="laser_frame_link">
+    <link name="${robot_name}/laser_frame_link">
       <visual>
         <origin
@@ -90,5 +90,5 @@
       </inertial>
     </link>
-    <gazebo reference="lidar_tower_link">
+    <gazebo reference="${robot_name}/lidar_tower_link">
       <material>Gazebo/DarkGrey</material>
     </gazebo>
@@ -99,5 +99,5 @@
       <disableFixedJointLumping>true</disableFixedJointLumping>
     </gazebo>
-    <gazebo reference="laser_frame_link">
+    <gazebo reference="${robot_name}/laser_frame_link">
       <material>Gazebo/DarkGrey</material>
       <sensor type="ray" name="rplidar">
@@ -128,8 +128,8 @@
         <plugin name="gazebo_ros_head_rplidar_controller" filename="libgazebo_ros_ray_sensor.so">
           <ros>
-            <remapping>~/out:=scan</remapping>
+            <remapping>~/out:=${robot_name}/scan</remapping>
           </ros>
           <output_type>sensor_msgs/LaserScan</output_type>
-          <frame_name>laser_frame_link</frame_name>
+          <frame_name>${robot_name}/laser_frame_link</frame_name>
         </plugin>
       </sensor>

File: src/rail_robot/urdf/plate.urdf.xacro (robot description, xacro)
@@ -5,9 +5,9 @@
       <xacro:insert_block name="origin"/>
       <parent
-        link="base_link"/>
+        link="${robot_name}/base_link"/>
       <child
-        link="plate_link"/>
+        link="${robot_name}/plate_link"/>
     </joint>
-    <link name="plate_link">
+    <link name="${robot_name}/plate_link">
       <visual>
         <origin
@@ -33,5 +33,5 @@
       <xacro:insert_block name="inertial"/>
     </link>
-    <gazebo reference="plate_link">
+    <gazebo reference="${robot_name}/plate_link">
       <material>Gazebo/DarkGrey</material>
     </gazebo>

File: src/rail_robot/urdf/rail_robot.urdf.xacro (robot description, xacro)
@@ -1,5 +1,6 @@
 <?xml version="1.0" ?>
 <robot name="rail_robot" xmlns:xacro="http://ros.org/wiki/xacro">
-  <xacro:property name="mesh_scale" value="0.001 0.001 0.001"/>
+  <xacro:arg name="robot_name"            default=""/>
+  <xacro:property name="robot_name" value="$(arg robot_name)"/>
   <material name="interbotix_black">
     <texture filename="package://rail_robot/media/materials/textures/interbotix_black.png"/>
@@ -9,54 +10,55 @@
   <xacro:include filename="$(find rail_robot)/urdf/battery.urdf.xacro" />
   <xacro:include filename="$(find rail_robot)/urdf/camera_tower.urdf.xacro" />
-  <xacro:include filename="$(find kobuki_description)/urdf/kobuki_standalone.urdf.xacro" />
-  <!-- Plate -->
-  <xacro:plate>
-    <origin
-      rpy="0 0 0"
-      xyz="0.0 0 0.08825"/>
-    <inertial>
+    <xacro:include filename="$(find rail_robot)/urdf/kobuki_version/locobot_kobuki.urdf.xacro"/>
+    <xacro:property name="mesh_scale" value="0.001 0.001 0.001"/>
+  <!-- ********************************** Plate **********************************  -->
+    <xacro:plate>
       <origin
         rpy="0 0 0"
-        xyz="0.050816 0 0.00475"/>
-      <mass value="0.571995"/>
-      <inertia
-        ixx="0.003115"
-        ixy="0"
-        ixz="0"
-        iyy="0.001813"
-        iyz="0"
-        izz="0.004919"/>
-    </inertial>
-  </xacro:plate>
-  <!-- Battery -->
-  <xacro:battery>
-    <origin
+        xyz="0.0 0 0.08825"/>
+      <inertial>
+        <origin
+          rpy="0 0 0"
+          xyz="0.050816 0 0.00475"/>
+        <mass value="0.571995"/>
+        <inertia
+          ixx="0.003115"
+          ixy="0"
+          ixz="0"
+          iyy="0.001813"
+          iyz="0"
+          izz="0.004919"/>
+      </inertial>
+    </xacro:plate>
+  <!-- ********************************** Battery **********************************  -->
+    <xacro:battery>
+      <origin
         rpy="0 0 0"
         xyz="-0.007 0 0.0125"/>
-  </xacro:battery>
-  <!-- Camera tower -->
-  <xacro:camera_tower>
-    <origin
-      rpy="0 0 0"
-      xyz="-0.023997 -0.000044 0.08823"/>
-    <inertial>
-      <origin
-        rpy="0 0 0"
-        xyz="-0.0372211000 -0.0026114300 0.1744600000"/>
-      <mass value="2.366224"/>
-      <inertia
-        ixx="0.0628500000"
-        ixy="0.0002152000"
-        ixz="0.0065630000"
-        iyy="0.0546000000"
-        iyz="-0.0004738000"
-        izz="0.0179300000"/>
-    </inertial>
-  </xacro:camera_tower>
-  <!-- lidar -->
-  <xacro:lidar>
-    <origin
-      rpy="0 0 0"
-      xyz="-0.074 0 0.44425"/>
-  </xacro:lidar>
+    </xacro:battery>
+  <!-- ********************************** Camera Tower **********************************  -->
+      <xacro:camera_tower>
+        <origin
+          rpy="0 0 0"
+          xyz="-0.023997 -0.000044 0.08823"/>
+        <inertial>
+          <origin
+            rpy="0 0 0"
+            xyz="-0.0372211000 -0.0026114300 0.1744600000"/>
+          <mass value="2.366224"/>
+          <inertia
+            ixx="0.0628500000"
+            ixy="0.0002152000"
+            ixz="0.0065630000"
+            iyy="0.0546000000"
+            iyz="-0.0004738000"
+            izz="0.0179300000"/>
+        </inertial>
+      </xacro:camera_tower>
+  <!-- ********************************** Lidar **********************************  -->
+        <xacro:lidar>
+          <origin
+            rpy="0 0 0"
+            xyz="-0.074 0 0.44425"/>
+        </xacro:lidar>
 </robot>
