Commit message: simulation working with ros2 control

File: src/rail_robot/urdf/kobuki_version/locobot_kobuki.urdf.xacro (robot description, xacro)
@@ -104,5 +104,5 @@
       link="${robot_name}/wheel_left_link"/>
   </joint>
-  <!-- <xacro:if value="${hardware_type == 'gz_classic'}">
+  <xacro:if value="${hardware_type == 'gz_classic'}">
     <ros2_control name="wheel_left_joint_controller" type="system">
       <hardware>
@@ -115,5 +115,5 @@
       </joint>
     </ros2_control>
-  </xacro:if> -->
+  </xacro:if>
   <link name="${robot_name}/wheel_left_link">
     <visual>
@@ -167,5 +167,5 @@
       link="${robot_name}/wheel_right_link"/>
   </joint>
-  <!-- <xacro:if value="${hardware_type == 'gz_classic'}">
+  <xacro:if value="${hardware_type == 'gz_classic'}">
     <ros2_control name="wheel_right_joint_controller" type="system">
       <hardware>
@@ -178,5 +178,5 @@
       </joint>
     </ros2_control>
-  </xacro:if> -->
+  </xacro:if>
   <link name="${robot_name}/wheel_right_link">
     <visual>
@@ -494,5 +494,5 @@
   </gazebo>
   <!-- Plugins -->
-  <!-- <gazebo>
+  <gazebo>
     <xacro:if value="${hardware_type == 'gz_classic'}">
       <plugin name="gazebo_ros2_control" filename="libgazebo_ros2_control.so">
@@ -502,13 +502,13 @@
         <robot_param>robot_description</robot_param>
         <robot_param_node>robot_state_publisher</robot_param_node>
-        <parameters> $(find interbotix_xslocobot_sim)/config/kobuki_version/$(arg robot_model)_controllers.yaml </parameters>
+        <parameters> $(find rail_robot)/config/ros2_control_sim.yaml </parameters>
       </plugin>
     </xacro:if>
     <xacro:if value="${hardware_type == 'gz_ignition'}">
       <plugin filename="ign_ros2_control-system" name="ign_ros2_control::IgnitionROS2ControlPlugin">
-        <parameters> $(find interbotix_xslocobot_sim)/config/kobuki_version/$(arg robot_model)_controllers.yaml </parameters>
+        <parameters> $(find interbotix_xslocobot_sim)/config/ros2_control_sim.yaml </parameters>
       </plugin>
     </xacro:if>
-    <plugin filename="libgazebo_ros_p3d.so" name="p3d_base_controller">
+    <!-- <plugin filename="libgazebo_ros_p3d.so" name="p3d_base_controller">
       <ros>
         <remapping>odom:=sim_ground_truth_pose</remapping>
@@ -521,5 +521,5 @@
       <rpy_offset>0.0 0.0 0.0</rpy_offset>
       <gaussian_noise>0</gaussian_noise>
-    </plugin>
-  </gazebo> -->
+    </plugin> -->
+  </gazebo>
 </robot>

File: src/rail_robot/urdf/rail_robot.urdf.xacro (robot description, xacro)
@@ -2,5 +2,7 @@
 <robot name="rail_robot" xmlns:xacro="http://ros.org/wiki/xacro">
   <xacro:arg name="robot_name"            default=""/>
+  <xacro:arg name="hardware_type"         default="gz_classic"/>
   <xacro:property name="robot_name" value="$(arg robot_name)"/>
+  <xacro:property name="hardware_type"    value="$(arg hardware_type)"/>
   <material name="interbotix_black">
     <texture filename="package://rail_robot/media/materials/textures/interbotix_black.png"/>

Commit message: drifting stops: fix gazebo reference in urdf

File: src/rail_robot/urdf/kobuki_version/locobot_kobuki.urdf.xacro (robot description, xacro)
@@ -82,5 +82,5 @@
     </inertial>
   </link>
-  <gazebo reference="base_link">
+  <gazebo reference="${robot_name}/base_link">
     <mu1>0.3</mu1>
     <mu2>0.3</mu2>
@@ -90,5 +90,5 @@
       <visualize>true</visualize>
       <contact>
-        <collision>base_footprint</collision>
+        <collision>${robot_name}/base_footprint</collision>
       </contact>
     </sensor>
@@ -149,5 +149,5 @@
     </inertial>
   </link>
-  <gazebo reference="wheel_left_link">
+  <gazebo reference="${robot_name}/wheel_left_link">
     <mu1>1.0</mu1>
     <mu2>1.0</mu2>
@@ -212,5 +212,5 @@
     </inertial>
   </link>
-  <gazebo reference="wheel_right_link">
+  <gazebo reference="${robot_name}/wheel_right_link">
     <mu1>1.0</mu1>
     <mu2>1.0</mu2>
@@ -253,5 +253,5 @@
     </inertial>
   </link>
-  <gazebo reference="caster_front_link">
+  <gazebo reference="${robot_name}/caster_front_link">
     <mu1>0.0</mu1>
     <mu2>0.0</mu2>
@@ -294,5 +294,5 @@
     </inertial>
   </link>
-  <gazebo reference="caster_back_link">
+  <gazebo reference="${robot_name}/caster_back_link">
     <mu1>0.0</mu1>
     <mu2>0.0</mu2>
@@ -326,5 +326,5 @@
     </inertial>
   </link>
-  <gazebo reference="gyro_link">
+  <gazebo reference="${robot_name}/gyro_link">
     <sensor name="imu" type="imu">
       <always_on>true</always_on>
@@ -375,5 +375,5 @@
     </inertial>
   </link>
-  <gazebo reference="cliff_sensor_left_link">
+  <gazebo reference="${robot_name}/cliff_sensor_left_link">
     <sensor name="cliff_sensor_left" type="ray">
       <always_on>true</always_on>
@@ -422,5 +422,5 @@
     </inertial>
   </link>
-  <gazebo reference="cliff_sensor_right_link">
+  <gazebo reference="${robot_name}/cliff_sensor_right_link">
     <sensor name="cliff_sensor_right" type="ray">
       <always_on>true</always_on>
@@ -469,5 +469,5 @@
     </inertial>
   </link>
-  <gazebo reference="cliff_sensor_front_link">
+  <gazebo reference="${robot_name}/cliff_sensor_front_link">
     <sensor name="cliff_sensor_front" type="ray">
       <always_on>true</always_on>
